Commit message: Add sensors, fix crash bug, cleanups

File: urdf/base.xacro (robot description, xacro)
@@ -1,22 +1,18 @@
 <?xml version="1.0"?>
 <robot xmlns:xacro="http://www.ros.org/wiki/xacro">
-  <!-- Loading some constants -->
   <xacro:include filename="$(find uuv_descriptions)/urdf/common.urdf.xacro"/>
-  <!-- Loading file with sensor macros -->
   <xacro:include filename="$(find uuv_sensor_ros_plugins)/urdf/sensor_snippets.xacro"/>
-  <!-- Loading the UUV simulator ROS plugin macros -->
   <xacro:include filename="$(find uuv_gazebo_ros_plugins)/urdf/snippets.xacro"/>
-  <!-- Loading vehicle's specific macros -->
   <xacro:include filename="$(find simulator)/urdf/snippets.xacro"/>
   <!--
-    Vehicle's parameters (remember to enter the model parameters below)
+       These figures are all taken from the default uuv simulator parameters.
+       Putting Nemo's values in did not work.
   -->
+  <!-- Parameters -->
   <xacro:property name="namespace" value="nemo"/>
   <xacro:property name="inertial_reference_frame" value="world"/>
-  <xacro:property name="mass" value="44.5"/>
-  <!-- Center of gravity -->
-  <xacro:property name="cog" value="0 0 0"/>
+  <xacro:property name="mass" value="1862.87"/>
   <!-- Fluid density -->
-  <xacro:property name="rho" value="1028"/>
+  <xacro:property name="rho" value="1028.0"/>
   <!--
     Visual mesh file for the vehicle, usually in DAE (Collada) format. Be sure to store the
@@ -26,9 +22,4 @@
   -->
   <xacro:property name="visual_mesh_file" value="file://$(find simulator)/meshes/nemo.dae"/>
-  <!-- Collision geometry mesh, usually in STL format (it is recommended to keep
-  this geometry as simple as possible to improve the performance the physics engine
-  regarding the computation of collision forces) -->
-  <!-- Unused, used simple box shape for collision instead -->
-  <!--xacro:property name="collision_mesh_file" value="file://$(find simulator)/meshes/nemo_collision.stl"/-->
   <!-- Vehicle macro -->
   <xacro:macro name="nemo_base" params="namespace *gazebo">
@@ -41,6 +32,6 @@
         <inertial>
           <mass value="${mass}" />
-          <origin xyz="${cog}" rpy="0 0 0"/>
-          <inertia ixx="1.69" ixy="-0.10" ixz="0.0" iyy="3.21" iyz="0.0" izz="2.94"/>
+          <origin xyz="0 0 0" rpy="0 0 0"/>
+          <inertia ixx="525.39" ixy="1.44" ixz="33.41" iyy="794.20" iyz="2.6" izz="691.23"/>
         </inertial>
         <visual>
@@ -62,7 +53,6 @@
     <!-- Set up hydrodynamic plugin given as input parameter -->
     <xacro:insert_block name="gazebo"/>
-    <!-- Include the thruster modules -->
+    <!-- Include the thruster and sensor modules -->
     <xacro:include filename="$(find simulator)/urdf/actuators.xacro"/>
-    <!-- Include the sensor modules -->
     <xacro:include filename="$(find simulator)/urdf/sensors.xacro"/>
   </xacro:macro>

File: urdf/gazebo.xacro (robot description, xacro)
@@ -2,11 +2,7 @@
 <robot xmlns:xacro="http://www.ros.org/wiki/xacro">
     <!-- Center of buoyancy -->
-    <xacro:property name="nemo_cob" value="0 0 0.14"/>
+    <xacro:property name="nemo_cob" value="0 0 0.3"/>
     <!-- Vehicle's actual volume (Gazebo cannot compute the volume out of the mesh) -->
-    <xacro:property name="nemo_volume" value="0.044"/>
-    <!-- Describing the dimensions of the vehicle's bounding box -->
-    <xacro:property name="nemo_length" value="0.9"/>
-    <xacro:property name="nemo_width"  value="0.6"/>
-    <xacro:property name="nemo_height" value="0.4"/>
+    <xacro:property name="nemo_volume" value="1.83826"/>
     <xacro:macro name="nemo_hydro_model" params="namespace">
       <!-- List of hydrodynamic models this robot's links -->
@@ -17,37 +13,30 @@
         <volume>${nemo_volume}</volume>
         <!-- Link's bounding box, it is used to recalculate the immersed
-        volume when close to the surface.
+        volume when close to the surface. These numbers are bs'ed.
         This is a workaround the invalid bounding box given by Gazebo-->
         <box>
-          <width>${nemo_width}</width>
-          <length>${nemo_length}</length>
-          <height>${nemo_height}</height>
+          <width>3.0</width>
+          <length>2.6</length>
+          <height>0.5</height>
         </box>
-        <!-- Center of buoyancy -->
         <center_of_buoyancy>${nemo_cob}</center_of_buoyancy>
-        <!-- Fossen's equation of motion -->
         <hydrodynamic_model>
           <type>fossen</type>
+          <!-- Added mass: see p.28 in Berg2012 -->
           <added_mass>
-            20 0  0  0  0  0
-            0  30 0  0  0  0
-            0  0  90 0  0  0
-            0  0  0  12 0  0
-            0  0  0  0  20 0
-            0  0  0  0  0  5
+               779.79 -6.8773 -103.32  8.5426 -165.54 -7.8033
+              -6.8773    1222   51.29  409.44 -5.8488  62.726
+              -103.32   51.29  3659.9  6.1112 -386.42  10.774
+               8.5426  409.44  6.1112   534.9 -10.027  21.019
+              -165.54 -5.8488 -386.42 -10.027  842.69 -1.1162
+              -7.8033  62.726  10.775  21.019 -1.1162  224.32
           </added_mass>
-          <!--
-            The linear damping coefficients can be provided as a diagonal (6 elements)
-            or a full matrix (36 coefficients), like the added-mass coefficients above
-          -->
+          <!-- Linear damping: see p.31 in Berg2012 -->
           <linear_damping>
-            -4 -10 -17.4 -6.4211 -8 -8
+              -74.82 -69.48 -728.4 -268.8 -309.77 -105
           </linear_damping>
-          <!--
-            The quadratic damping coefficients can be provided as a diagonal (6 elements)
-            or a full matrix (36 coefficients), like the added-mass coefficients above
-          -->
+          <!-- Non-linear damping: see p.30 in Berg2012 -->
           <quadratic_damping>
-            -10 -23.709 -43.500 -16.053 -18.500 -18.500
+              -748.22 -992.53 -1821.01 -672 -774.44 -523.27
           </quadratic_damping>
         </hydrodynamic_model>

File: urdf/sensors.xacro (robot description, xacro)
@@ -61,7 +61,30 @@
   <link name="${namespace}/down_camera_link"/>
   <joint name="${namespace}/down_camera_joint" type="fixed">
-    <origin xyz="0 0.19 -0.17" rpy="0 1.5707 0" />
+    <origin xyz="0 0.19 -0.17" rpy="0 ${0.5*pi} 0" />
     <parent link="${namespace}/base_link" />
     <child link="${namespace}/down_camera_link" />
   </joint>
+  <!-- DVL sensor -->
+  <xacro:custom_dvl
+    namespace="${namespace}"
+    suffix=""
+    parent_link="${namespace}/base_link"
+    topic="dvl"
+    noise_sigma="0"
+    noise_amplitude="0"
+    update_rate="10"
+    reference_frame="world">
+    <origin xyz="-0.08 0.0 -0.17" rpy="0 ${0.5*pi} 0" />
+  </xacro:custom_dvl>
+  <!-- IMU  -->
+  <xacro:default_imu_macro
+    namespace="${namespace}"
+    parent_link="${namespace}/base_link"
+    inertial_reference_frame="${inertial_reference_frame}">
+    <origin xyz="0 0 0" rpy="0 0 0"/>
+  </xacro:default_imu_macro>
+  <!-- Pressure  -->
+  <xacro:default_pressure_macro namespace="${namespace}" parent_link="${namespace}/base_link">
+    <origin xyz="-0.08 0.0 0.2" rpy="0 0 0"/>
+  </xacro:default_pressure_macro>
 </robot>

File: urdf/snippets.xacro (robot description, xacro)
@@ -1,89 +1,122 @@
 <?xml version="1.0"?>
 <robot xmlns:xacro="http://www.ros.org/wiki/xacro">
-  <!--                                                                      -->
-  <!-- MACRO FOR THRUSTER UNITS  -->
-  <!--                                                                      -->
-  <!-- Provide the propeller mesh in a separate file with the rotation axis
-  over propeller's frame X-axis in DAE (Collada) or STL format.
-  -->
-  <xacro:property name="prop_mesh_file" value="file://$(find simulator)/meshes/propeller.dae"/>
-  <!--
-    Thruster macro with integration of joint and link. The thrusters should
-    be initialized in the actuators.xacro file.
-  -->
-  <xacro:macro name="thruster_macro" params="robot_namespace thruster_id *origin">
-    <!--
-    Dummy link as place holder for the thruster frame,
-    since thrusters can often be inside the collision geometry
-    of the vehicle and may cause internal collisions if set otherwise
-    -->
-    <link name="${robot_namespace}/thruster_${thruster_id}">
-      <visual>
-        <geometry>
-          <mesh filename="${prop_mesh_file}" scale="1 1 1" />
-        </geometry>
-      </visual>
+  <!-- Thruster joint and link class -->
+  <xacro:macro name="thruster_macro"
+    params="robot_namespace thruster_id *origin">
+    <xacro:thruster_module_first_order_basic_fcn_macro
+      namespace="${robot_namespace}"
+      thruster_id="${thruster_id}"
+      mesh_filename="file://$(find simulator)/meshes/propeller.dae"
+      dyn_time_constant="0.01"
+      rotor_constant="0.00031">
+      <xacro:insert_block name="origin"/>
+    </xacro:thruster_module_first_order_basic_fcn_macro>
+  </xacro:macro>
+  <!-- Setup Individual DVL Ray Class -->
+  <xacro:macro name="custom_dvl_ray" params="namespace suffix index pitch yaw update_rate">
+    <link name="${namespace}/dvl${suffix}_sonar${index}_link">
       <inertial>
-        <mass value="0.001" />
-        <origin xyz="0 0 0" rpy="0 0 0"/>
-        <inertia ixx="0.000000017" ixy="0.0" ixz="0.0"
-               iyy="0.000000017" iyz="0.0"
-               izz="0.000000017" />
+        <mass value="0.001" />  <!-- [kg] -->
+        <origin xyz="0 0 0" rpy="0 0 0" />
+        <inertia ixx="0.000000017" ixy="0" ixz="0" iyy="0.000000017" iyz="0" izz="0.000000017" />
       </inertial>
+      <xacro:no_collision/>
     </link>
-    <!-- Joint between thruster link and vehicle base link -->
-    <joint name="${robot_namespace}/thruster_${thruster_id}_joint" type="continuous">
+    <joint name="${namespace}/dvl${suffix}_sonar${index}_joint" type="revolute">
+      <origin xyz="0 0 0" rpy="0 ${pitch} ${yaw}"/>
+      <parent link="${namespace}/dvl${suffix}_link" />
+      <child link="${namespace}/dvl${suffix}_sonar${index}_link" />
+      <limit upper="0" lower="0" effort="0" velocity="0" />
+      <axis xyz="1 0 0"/>
+    </joint>
+    <gazebo reference="${namespace}/dvl${suffix}_sonar${index}_link">
+      <sensor type="ray" name="dvl${suffix}_sonar${index}">
+        <pose>0 0 0 0 0 0</pose>
+        <update_rate>${update_rate}</update_rate>
+        <visualize>false</visualize>
+        <ray>
+          <scan>
+            <horizontal>
+              <samples>1</samples>
+              <resolution>1</resolution>
+              <min_angle>0</min_angle>
+              <max_angle>0</max_angle>
+            </horizontal>
+          </scan>
+          <range>
+            <min>0.2</min>
+            <max>81</max>
+            <resolution>0.01</resolution>
+          </range>
+        </ray>
+        <plugin filename="libgazebo_ros_range.so" name="dvl${suffix}_sonar${index}">
+          <gaussianNoise>0.005</gaussianNoise>
+          <alwaysOn>true</alwaysOn>
+          <updateRate>${update_rate}</updateRate>
+          <topicName>${topic}_sonar${index}</topicName>
+          <frameName>${namespace}/dvl${suffix}_sonar${index}_link</frameName>
+          <fov>0.06</fov>
+          <radiation>ultrasound</radiation>
+        </plugin>
+      </sensor>
+    </gazebo>
+  </xacro:macro>
+  <!-- Setup Custom DVL class -->
+  <xacro:macro name="custom_dvl"
+    params="namespace suffix parent_link topic *origin update_rate
+    reference_frame noise_sigma noise_amplitude">
+    <link name="${namespace}/dvl${suffix}_link">
+      <inertial>
+        <mass value="0.001" />  <!-- [kg] -->
+        <origin xyz="0 0 0" rpy="0 0 0" />
+        <inertia ixx="0.000000017" ixy="0" ixz="0" iyy="0.000000017" iyz="0" izz="0.000000017" />
+      </inertial>
+      <xacro:no_collision/>
+    </link>
+    <joint name="${namespace}/dvl${suffix}_joint" type="revolute">
       <xacro:insert_block name="origin" />
-      <axis xyz="1 0 0" />
-      <parent link="${robot_namespace}/base_link" />
-      <child link="${robot_namespace}/thruster_${thruster_id}" />
+      <parent link="${parent_link}" />
+      <child link="${namespace}/dvl${suffix}_link" />
+      <limit upper="0" lower="0" effort="0" velocity="0" />
+      <axis xyz="1 0 0"/>
     </joint>
+    <xacro:custom_dvl_ray
+      namespace="${namespace}" suffix=""
+      index="0" pitch="-0.52" yaw="0.0" update_rate="${update_rate}">
+    </xacro:custom_dvl_ray>
+    <xacro:custom_dvl_ray
+      namespace="${namespace}" suffix=""
+      index="1" pitch="0" yaw="0.52" update_rate="${update_rate}">
+    </xacro:custom_dvl_ray>
+    <xacro:custom_dvl_ray
+      namespace="${namespace}" suffix=""
+      index="2" pitch="0.52" yaw="0.0" update_rate="${update_rate}">
+    </xacro:custom_dvl_ray>
+    <xacro:custom_dvl_ray
+      namespace="${namespace}" suffix=""
+      index="3" pitch="0.0" yaw="-0.52" update_rate="${update_rate}">
+    </xacro:custom_dvl_ray>
     <gazebo>
-      <!-- Thruster ROS plugin -->
-      <plugin name="${robot_namespace}_${thruster_id}_thruster_model" filename="libuuv_thruster_ros_plugin.so">
-        <!-- Name of the thruster link -->
-        <linkName>${robot_namespace}/thruster_${thruster_id}</linkName>
-        <!-- Name of the joint between thruster and vehicle base link -->
-        <jointName>${robot_namespace}/thruster_${thruster_id}_joint</jointName>
-        <!-- Make the thruster aware of its id -->
-        <thrusterID>${thruster_id}</thrusterID>
-        <!--
-        Value from 0 to 1 to set the efficiency of the output thrust force
-        Default value is 1.0
-        -->
-        <thrust_efficiency>1</thrust_efficiency>
-        <!--
-        Value from 0 to 1 to set the efficiency of the propeller as a factor
-        to be multiplied to the current value of the state variable at each
-        iteration.
-        Default value is 1.0
-        -->
-        <propeller_efficiency>1</propeller_efficiency>
-        <!--
-        Choose one of the propeller dynamics models below for your implementation
-        This will describe the dynamic model for the state variable of your thruster unit,
-        which can be, e.g., the angular velocity of the propeller.
-        -->
-        <dynamics>
-          <type>FirstOrder</type>
-          <timeConstant>0.01</timeConstant>
-        </dynamics>
-        <!--
-        Choose one of the model for the steady-state curve describing the
-        relationship between the state variable and the output thrust force
-        -->
-        <!-- 1) Basic curve
-        Input: x
-        Output: thrust
-        Function: thrust = rotorConstant * x * abs(x)
-        -->
-        <conversion>
-          <type>Basic</type>
-          <rotorConstant>0.00031</rotorConstant>
-        </conversion>
+      <plugin filename="libuuv_gazebo_ros_dvl_plugin.so" name="libuuv_gazebo_dvl${suffix}_plugin">
+        <robot_namespace>${namespace}</robot_namespace> <!-- (string, required): ros namespace in which the messages are published -->
+        <link_name>${namespace}/dvl${suffix}_link</link_name> <!-- (string, required): name of the body which holds the IMU sensor -->
+        <sensor_topic>${topic}</sensor_topic> <!-- (string): name of the sensor output topic and prefix of service names -->
+        <update_rate>${update_rate}</update_rate> <!-- Update period [s] -->
+        <noise_sigma>${noise_sigma}</noise_sigma> <!-- std dev of position estimates in x, y, z [m/s] -->
+        <noise_amplitude>${noise_amplitude}</noise_amplitude>
+        <enable_gazebo_messages>false</enable_gazebo_messages>
+        <enable_local_ned_frame>false</enable_local_ned_frame>
+        <static_reference_frame>${reference_frame}</static_reference_frame>
+        <!-- Declaring the beams -->
+        <beam_link_name_0>${namespace}/dvl_sonar0_link</beam_link_name_0>
+        <beam_link_name_1>${namespace}/dvl_sonar1_link</beam_link_name_1>
+        <beam_link_name_2>${namespace}/dvl_sonar2_link</beam_link_name_2>
+        <beam_link_name_3>${namespace}/dvl_sonar3_link</beam_link_name_3>
+        <!-- Declaring the beam output topics -->
+        <beam_topic_0>${topic}_sonar0</beam_topic_0>
+        <beam_topic_1>${topic}_sonar1</beam_topic_1>
+        <beam_topic_2>${topic}_sonar2</beam_topic_2>
+        <beam_topic_3>${topic}_sonar3</beam_topic_3>
       </plugin>
-    </gazebo>
-    <gazebo reference="${robot_namespace}/thruster_${thruster_id}">
-      <selfCollide>false</selfCollide>
     </gazebo>
   </xacro:macro>
