Commit message: Add new nemo model from Sri

File: urdf/actuators.xacro (robot description, xacro)
@@ -11,26 +11,26 @@
     <!-- Order of thrusterse is VERT FL, VERT FR, VERT BL, VERT BR, SURGE FL, SURGE FR, SURGE BL, SURGE BR -->
     <xacro:thruster_macro robot_namespace="${namespace}" thruster_id="0">
-        <origin rpy="0 -1.57 0" xyz="0.263 0.215 0.14"/>
+        <origin rpy="0 -1.57 0" xyz="0.341 0.215 -0.06"/>
     </xacro:thruster_macro>
     <xacro:thruster_macro robot_namespace="${namespace}" thruster_id="1">
-        <origin rpy="0 -1.57 0" xyz="0.263 -0.215 0.14"/>
+        <origin rpy="0 -1.57 0" xyz="0.341 -0.215 -0.06"/>
     </xacro:thruster_macro>
     <xacro:thruster_macro robot_namespace="${namespace}" thruster_id="2">
-        <origin rpy="0 -1.57 0" xyz="-0.24 0.215 0.14"/>
+        <origin rpy="0 -1.57 0" xyz="-0.1635 0.215 -0.06"/>
     </xacro:thruster_macro>
     <xacro:thruster_macro robot_namespace="${namespace}" thruster_id="3">
-        <origin rpy="0 -1.57 0" xyz="-0.24 -0.215 0.14"/>
+        <origin rpy="0 -1.57 0" xyz="-0.1635 -0.215 -0.06"/>
     </xacro:thruster_macro>
     <xacro:thruster_macro robot_namespace="${namespace}" thruster_id="4">
-        <origin rpy="0 0 2.36" xyz="0.38 0.25 -0.05"/>
+        <origin rpy="0 0 2.36" xyz="0.45 0.26 -0.27"/>
     </xacro:thruster_macro>
     <xacro:thruster_macro robot_namespace="${namespace}" thruster_id="5">
-        <origin rpy="0 0 -2.36" xyz="0.38 -0.25 -0.05"/>
+        <origin rpy="0 0 -2.36" xyz="0.45 -0.26 -0.27"/>
     </xacro:thruster_macro>
     <xacro:thruster_macro robot_namespace="${namespace}" thruster_id="6">
-        <origin rpy="0 0 -2.36" xyz="-0.359 0.25 -0.05"/>
+        <origin rpy="0 0 -2.36" xyz="-0.3 0.23 -0.27"/>
     </xacro:thruster_macro>
     <xacro:thruster_macro robot_namespace="${namespace}" thruster_id="7">
-        <origin rpy="0 0 2.36" xyz="-0.359 -0.25 -0.05"/>
+        <origin rpy="0 0 2.36" xyz="-0.3 -0.23 -0.27"/>
     </xacro:thruster_macro>
 </robot>

File: urdf/sensors.xacro (robot description, xacro)
@@ -29,5 +29,5 @@
   <link name="${namespace}/front_camera_link"/>
   <joint name="${namespace}/front_camera_joint" type="fixed">
-    <origin xyz="0.39 0 -0.05" rpy="0 0 0" />
+    <origin xyz="0.46 0 -0.27" rpy="0 0 0" />
     <parent link="${namespace}/base_link" />
     <child link="${namespace}/front_camera_link" />
@@ -61,5 +61,5 @@
   <link name="${namespace}/down_camera_link"/>
   <joint name="${namespace}/down_camera_joint" type="fixed">
-    <origin xyz="0 0.19 -0.17" rpy="0 ${0.5*pi} 0" />
+    <origin xyz="-0.018 0.218 -0.37" rpy="0 ${0.5*pi} 0" />
     <parent link="${namespace}/base_link" />
     <child link="${namespace}/down_camera_link" />
@@ -75,5 +75,5 @@
     update_rate="10"
     reference_frame="world">
-    <origin xyz="-0.08 0.0 -0.17" rpy="0 ${0.5*pi} 0" />
+    <origin xyz="-0.003 0.0 -0.39" rpy="0 ${0.5*pi} 0" />
   </xacro:custom_dvl>
   <!-- IMU  -->
@@ -86,5 +86,5 @@
   <!-- Pressure  -->
   <xacro:default_pressure_macro namespace="${namespace}" parent_link="${namespace}/base_link">
-    <origin xyz="-0.08 0.0 0.2" rpy="0 0 0"/>
+    <origin xyz="0 0 0" rpy="0 0 0"/>
   </xacro:default_pressure_macro>
 </robot>

Commit message: Update nemo model, fix parameters

File: urdf/actuators.xacro (robot description, xacro)
@@ -11,26 +11,26 @@
     <!-- Order of thrusterse is VERT FL, VERT FR, VERT BL, VERT BR, SURGE FL, SURGE FR, SURGE BL, SURGE BR -->
     <xacro:thruster_macro robot_namespace="${namespace}" thruster_id="0">
-        <origin rpy="0 -1.57 0" xyz="0.341 0.215 -0.06"/>
+        <origin rpy="0 -1.57 0" xyz="0.341 0.215 0.18"/>
     </xacro:thruster_macro>
     <xacro:thruster_macro robot_namespace="${namespace}" thruster_id="1">
-        <origin rpy="0 -1.57 0" xyz="0.341 -0.215 -0.06"/>
+        <origin rpy="0 -1.57 0" xyz="0.341 -0.215 0.18"/>
     </xacro:thruster_macro>
     <xacro:thruster_macro robot_namespace="${namespace}" thruster_id="2">
-        <origin rpy="0 -1.57 0" xyz="-0.1635 0.215 -0.06"/>
+        <origin rpy="0 -1.57 0" xyz="-0.1635 0.215 0.18"/>
     </xacro:thruster_macro>
     <xacro:thruster_macro robot_namespace="${namespace}" thruster_id="3">
-        <origin rpy="0 -1.57 0" xyz="-0.1635 -0.215 -0.06"/>
+        <origin rpy="0 -1.57 0" xyz="-0.1635 -0.215 0.18"/>
     </xacro:thruster_macro>
     <xacro:thruster_macro robot_namespace="${namespace}" thruster_id="4">
-        <origin rpy="0 0 2.36" xyz="0.45 0.26 -0.27"/>
+        <origin rpy="0 0 2.36" xyz="0.45 0.26 0"/>
     </xacro:thruster_macro>
     <xacro:thruster_macro robot_namespace="${namespace}" thruster_id="5">
-        <origin rpy="0 0 -2.36" xyz="0.45 -0.26 -0.27"/>
+        <origin rpy="0 0 -2.36" xyz="0.45 -0.26 0"/>
     </xacro:thruster_macro>
     <xacro:thruster_macro robot_namespace="${namespace}" thruster_id="6">
-        <origin rpy="0 0 -2.36" xyz="-0.3 0.23 -0.27"/>
+        <origin rpy="0 0 -2.36" xyz="-0.3 0.23 0"/>
     </xacro:thruster_macro>
     <xacro:thruster_macro robot_namespace="${namespace}" thruster_id="7">
-        <origin rpy="0 0 2.36" xyz="-0.3 -0.23 -0.27"/>
+        <origin rpy="0 0 2.36" xyz="-0.3 -0.23 0"/>
     </xacro:thruster_macro>
 </robot>

File: urdf/sensors.xacro (robot description, xacro)
@@ -29,5 +29,5 @@
   <link name="${namespace}/front_camera_link"/>
   <joint name="${namespace}/front_camera_joint" type="fixed">
-    <origin xyz="0.46 0 -0.27" rpy="0 0 0" />
+    <origin xyz="0.46 0 0" rpy="0 0 0" />
     <parent link="${namespace}/base_link" />
     <child link="${namespace}/front_camera_link" />
@@ -59,7 +59,9 @@
     </sensor>
   </gazebo>
+  <!-- The down camera location is put lower than usual because otherewise the landing gear
+       takes up a large part of the down camera image -->
   <link name="${namespace}/down_camera_link"/>
   <joint name="${namespace}/down_camera_joint" type="fixed">
-    <origin xyz="-0.018 0.218 -0.37" rpy="0 ${0.5*pi} 0" />
+    <origin xyz="-0.018 0.218 -0.155" rpy="0 ${0.5*pi} 0" />
     <parent link="${namespace}/base_link" />
     <child link="${namespace}/down_camera_link" />
@@ -75,5 +77,5 @@
     update_rate="10"
     reference_frame="world">
-    <origin xyz="-0.003 0.0 -0.39" rpy="0 ${0.5*pi} 0" />
+    <origin xyz="-0.003 0.0 -0.1" rpy="0 ${0.5*pi} 0" />
   </xacro:custom_dvl>
   <!-- IMU  -->
